Commit message: final

File: dual_arm_demo/urdf/dual_arm_scene.xacro (robot description, xacro)
@@ -4,9 +4,9 @@
     <xacro:include filename="$(find dual_arm_demo)/urdf/groot.xacro" />
     <link name="world" />
-    <xacro:rocket parent="world" >
-        <origin xyz="0 1 1" rpy="0 0 0" />
+    <xacro:rocket parent="world">
+        <origin xyz="0 0.5 1" rpy="0 0 0" />
     </xacro:rocket>
-    <xacro:groot parent="world" >
-        <origin xyz="0 -1 1" rpy="0 0 0" />
+    <xacro:groot parent="world">
+        <origin xyz="0 -0.5 1" rpy="0 0 0" />
     </xacro:groot>
 </robot>
